Commit message: turtlebot2 sim update

File: turtlebot2/turtlebot2/urdf/colors.urdf.xacro (robot description, xacro)
@@ -16,11 +16,15 @@
   <xacro:create_color name="DarkGray" value="0.1 0.1 0.1 0.5"/>
   <xacro:create_color name="Black" value="0 0 0 1"/>
-  <xacro:gazebo_color link="tick1_link" color="Gray"/>
-  <xacro:gazebo_color link="tick2_link" color="Gray"/>
-  <xacro:gazebo_color link="tick3_link" color="Gray"/>
-  <xacro:gazebo_color link="tick4_link" color="Gray"/>
-  <xacro:gazebo_color link="tick5_link" color="Gray"/>
+  <xacro:gazebo_color link="base_tick1_link" color="Gray"/>
+  <xacro:gazebo_color link="base_tick2_link" color="Gray"/>
+  <xacro:gazebo_color link="base_tick3_link" color="Gray"/>
+  <xacro:gazebo_color link="base_tick4_link" color="Gray"/>
+  <xacro:gazebo_color link="base_tick5_link" color="Gray"/>
+  <xacro:gazebo_color link="camera_support_tick1_link" color="Gray"/>
+  <xacro:gazebo_color link="camera_support_tick2_link" color="Gray"/>
+  <xacro:gazebo_color link="lower_base_link" color="DarkGrey"/>
   <xacro:gazebo_color link="middle_base_link" color="DarkGrey"/>
-  <xacro:gazebo_color link="laser_base_link" color="DarkGrey"/>
+  <xacro:gazebo_color link="upper_base_link" color="DarkGrey"/>
+  <xacro:gazebo_color link="camera_support_base_link" color="DarkGrey"/>
   <xacro:gazebo_color link="camera_link" color="Black"/>
   <xacro:gazebo_color link="lidar_link" color="Black"/>

File: turtlebot2/turtlebot2/urdf/structures.urdf.xacro (robot description, xacro)
@@ -28,3 +28,28 @@
     </joint>
   </xacro:macro>
+  <xacro:macro name="cube_structure" params="name x y z x_size y_size z_size parent">
+    <link name="${name}_link">
+      <visual>
+        <origin xyz="0 0 0" rpy="0 0 0"/>
+        <geometry>
+          <box size="${x_size} ${y_size} ${z_size}"/>
+        </geometry>
+      </visual>
+      <collision name="base">
+        <origin xyz="0 0 0" rpy="0 0 0"/>
+        <geometry>
+          <box size="${x_size} ${y_size} ${z_size}"/>
+        </geometry>
+      </collision>
+      <inertial>
+        <mass value="0.3"/>
+        <inertia  ixx="1.0" ixy="0.0"  ixz="0.0"  iyy="100.0"  iyz="0.0"  izz="1.0" />
+      </inertial>
+    </link>
+    <joint name="${name}_joint" type="fixed">
+      <origin xyz="${x} ${y} ${z}" rpy="0 0 0"/>
+      <parent link="${parent}"/>
+      <child link="${name}_link" />
+    </joint>
+  </xacro:macro>
 </robot>

File: turtlebot2/turtlebot2/urdf/turtlebot2.urdf (robot description, URDF)
Before this commit: robot turtlebot2, 20 links, 19 joints
Links:
- removed link laser_base_link
- removed link tick1_link
- removed link tick2_link
- removed link tick3_link
- removed link tick4_link
- removed link tick5_link
- added link base_tick1_link, mass 0.3; collision cylinder length=0.35 radius=0.005; visual cylinder length=0.35 radius=0.005
- added link base_tick2_link, mass 0.3; collision cylinder length=0.35 radius=0.005; visual cylinder length=0.35 radius=0.005
- added link base_tick3_link, mass 0.3; collision cylinder length=0.35 radius=0.005; visual cylinder length=0.35 radius=0.005
- added link base_tick4_link, mass 0.3; collision cylinder length=0.35 radius=0.005; visual cylinder length=0.35 radius=0.005
- added link base_tick5_link, mass 0.3; collision cylinder length=0.15 radius=0.005; visual cylinder length=0.15 radius=0.005
- added link camera_support_base_link, mass 0.3; collision box size=0.0175 0.15 0.005; visual box size=0.0175 0.15 0.005
- added link camera_support_tick1_link, mass 0.3; collision cylinder length=0.1 radius=0.005; visual cylinder length=0.1 radius=0.005
- added link camera_support_tick2_link, mass 0.3; collision cylinder length=0.1 radius=0.005; visual cylinder length=0.1 radius=0.005
- added link lower_base_link, mass 0.3; collision cylinder length=0.01 radius=0.18; visual cylinder length=0.01 radius=0.18
- added link upper_base_link, mass 0.3; collision cylinder length=0.01 radius=0.18; visual cylinder length=0.01 radius=0.18
Joints:
- removed joint laser_base_joint
- removed joint tick1_joint
- removed joint tick2_joint
- removed joint tick3_joint
- removed joint tick4_joint
- removed joint tick5_joint
- added joint base_tick1_joint: type fixed, parent base_link, child base_tick1_link, origin xyz=0.08 0.14 0.25 rpy=0 0 0
- added joint base_tick2_joint: type fixed, parent base_link, child base_tick2_link, origin xyz=-0.09 0.12 0.25 rpy=0 0 0
- added joint base_tick3_joint: type fixed, parent base_link, child base_tick3_link, origin xyz=-0.09 -0.12 0.25 rpy=0 0 0
- added joint base_tick4_joint: type fixed, parent base_link, child base_tick4_link, origin xyz=0.08 -0.14 0.25 rpy=0 0 0
- added joint base_tick5_joint: type fixed, parent base_link, child base_tick5_link, origin xyz=0.15 0.0 0.14 rpy=0 0 0
- added joint camera_support_base_joint: type fixed, parent middle_base_link, child camera_support_base_link, origin xyz=0.13 0 0.0975 rpy=0 0 0
- added joint camera_support_tick1_joint: type fixed, parent middle_base_link, child camera_support_tick1_link, origin xyz=0.13 0.05 0.05 rpy=0 0 0
- added joint camera_support_tick2_joint: type fixed, parent middle_base_link, child camera_support_tick2_link, origin xyz=0.13 -0.05 0.05 rpy=0 0 0
- added joint lower_base_joint: type fixed, parent base_link, child lower_base_link, origin xyz=0.0 0.0 0.155 rpy=0 0 0
- added joint upper_base_joint: type fixed, parent base_link, child upper_base_link, origin xyz=0.0 0.0 0.42 rpy=0 0 0
- joint lidar_joint: parent laser_base_link -> upper_base_link
- joint middle_base_joint: origin xyz=0.0 0.0 0.25 rpy=0 0 0 -> xyz=0.0 0.0 0.208 rpy=0 0 0

File: turtlebot2/turtlebot2/urdf/turtlebot2.urdf.xacro (robot description, xacro)
@@ -6,12 +6,16 @@
   <xacro:include filename="$(find turtlebot2)/urdf/structures.urdf.xacro"/>
   <xacro:include filename="$(find turtlebot2)/urdf/colors.urdf.xacro"/>
-  <xacro:cylinder_structure name="tick1" x="0.08" y="0.14" z="0.2" length="0.33" radius="0.005" parent="base_link"/>
-  <xacro:cylinder_structure name="tick2" x="-0.09" y="0.12" z="0.2" length="0.33" radius="0.005" parent="base_link"/>
-  <xacro:cylinder_structure name="tick3" x="-0.09" y="-0.12" z="0.2" length="0.33" radius="0.005" parent="base_link"/>
-  <xacro:cylinder_structure name="tick4" x="0.08" y="-0.14" z="0.2" length="0.33" radius="0.005" parent="base_link"/>
-  <xacro:cylinder_structure name="tick5" x="-0.15" y="0.0" z="0.2" length="0.33" radius="0.005" parent="base_link"/>
-  <xacro:cylinder_structure name="laser_base" x="0.0" y="0.0" z="0.35" length="0.01" radius="0.18" parent="base_link"/>
-  <xacro:cylinder_structure name="middle_base" x="0.0" y="0.0" z="0.25" length="0.01" radius="0.18" parent="base_link"/>
+  <xacro:cylinder_structure name="base_tick1" x="0.08" y="0.14" z="0.25" length="0.35" radius="0.005" parent="base_link"/>
+  <xacro:cylinder_structure name="base_tick2" x="-0.09" y="0.12" z="0.25" length="0.35" radius="0.005" parent="base_link"/>
+  <xacro:cylinder_structure name="base_tick3" x="-0.09" y="-0.12" z="0.25" length="0.35" radius="0.005" parent="base_link"/>
+  <xacro:cylinder_structure name="base_tick4" x="0.08" y="-0.14" z="0.25" length="0.35" radius="0.005" parent="base_link"/>
+  <xacro:cylinder_structure name="base_tick5" x="0.15" y="0.0" z="0.14" length="0.15" radius="0.005" parent="base_link"/>
+  <xacro:cylinder_structure name="camera_support_tick1" x="0.13" y="0.05" z="0.05" length="0.1" radius="0.005" parent="middle_base_link"/>
+  <xacro:cylinder_structure name="camera_support_tick2" x="0.13" y="-0.05" z="0.05" length="0.1" radius="0.005" parent="middle_base_link"/>
+  <xacro:cylinder_structure name="lower_base" x="0.0" y="0.0" z="0.155" length="0.01" radius="0.18" parent="base_link"/>
+  <xacro:cylinder_structure name="middle_base" x="0.0" y="0.0" z="0.208" length="0.01" radius="0.18" parent="base_link"/>
+  <xacro:cylinder_structure name="upper_base" x="0.0" y="0.0" z="0.42" length="0.01" radius="0.18" parent="base_link"/>
+  <xacro:cube_structure name="camera_support_base" x="0.13" y="0" z="0.0975" x_size="0.0175" y_size="0.15" z_size="0.005" parent="middle_base_link"/>
   <xacro:set_camera name="camera" xyz="0.13 0 0.32" rpy="0 0 0" parent_frame="base_link"/>
-  <xacro:set_lidar name="lidar" xyz="0 0 0.0275" parent_frame="laser_base_link"/>
+  <xacro:set_lidar name="lidar" xyz="0 0 0.0275" parent_frame="upper_base_link"/>
 </robot>
